File: TTRV PCB V5/ThinkTankTimerVote.kicad_sch (KiCad schematic)
At the start: 22 parts, among them J1 BattLeft, J2 Conn_01x02, J4 Conn_01x04, Q1 IRLML2060, SW1 SW_DPDT_x2, SW2 SW_Push, SW3 SW_Push, SW4 SW_Push, U2 HT75xx-1-SOT89, U3 LTC4054ES5-4.2

Commit message: Update PCB
Parts:
- added R9: 20k, Resistor_SMD:R_0603_1608Metric, symbol Device:R
- added R9: 10k, Resistor_SMD:R_0603_1608Metric, symbol Device:R
- C6, C9: footprint Capacitor_SMD:C_0402_1005Metric -> Capacitor_SMD:C_0603_1608Metric
- D2: footprint LED_SMD:LED_0603_1608Metric -> LED_SMD:LED_0805_2012Metric
- R14, R8, R9: footprint Resistor_SMD:R_0402_1005Metric -> Resistor_SMD:R_0603_1608Metric
Connections:
- net Batt+: now also R9.2
- net GND: now also R9.1
- net ADC1_BAT: now reaches U1.1 (GPIO1)
- net ADC1_BAT: now also R9.1, R9.2
Other:
- note added: "Measure Battery Charge"
Changed lines of the file:
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@@
   (junction (at 179.07 121.92) (diameter 0) (color 0 0 0 0)
   )
+  (junction (at 132.08 175.26) (diameter 0) (color 0 0 0 0)
+  )
   (junction (at 223.52 113.03) (diameter 0) (color 0 0 0 0)
   )
@@
     (stroke (width 0) (type default))
   )
+  (wire (pts (xy 124.46 185.42) (xy 124.46 182.88))
+    (stroke (width 0) (type default))
+  )
   (wire (pts (xy 233.68 123.19) (xy 240.03 123.19))
     (stroke (width 0) (type default))
   )
+  (wire (pts (xy 132.08 175.26) (xy 139.7 175.26))
+    (stroke (width 0) (type default))
+  )
   (wire (pts (xy 234.95 73.66) (xy 232.41 73.66))
     (stroke (width 0) (type default))
@@
     (stroke (width 0) (type default))
   )
+  (wire (pts (xy 132.08 171.45) (xy 132.08 175.26))
+    (stroke (width 0) (type default))
+  )
   (wire (pts (xy 199.39 54.61) (xy 190.5 54.61))
     (stroke (width 0) (type default))
@@
     (stroke (width 0) (type default))
   )
+  (wire (pts (xy 124.46 175.26) (xy 132.08 175.26))
+    (stroke (width 0) (type default))
+  )
   (wire (pts (xy 186.69 134.62) (xy 186.69 127))
     (stroke (width 0) (type default))
@@
     (stroke (width 0) (type default))
   )
+  (rectangle (start 107.95 162.56) (end 168.91 194.31)
+    (stroke (width 0) (type default))
+    (fill (type none))
+  )
   (rectangle (start 222.25 54.61) (end 257.81 81.28)
     (stroke (width 0) (type default))
@@
     (stroke (width 0) (type default))
     (fill (type none))
+  )
+  (text "Measure Battery Charge" (at 110.49 167.64 0)
+    (effects (font (size 2.27 2.27)) (justify left bottom))
   )
   (text "tested and working\n4-23-2024" (at 182.88 106.68 0)
@@
     )
   )
+  (global_label "ADC1_BAT" (shape input) (at 132.08 171.45 0) (fields_autoplaced)
+    (effects (font (size 1.27 1.27)) (justify left))
+    (property "Intersheetrefs" "${INTERSHEET_REFS}" (at 144.1971 171.45 0)
+      (effects (font (size 1.27 1.27)) (justify left) hide)
+    )
+  )
   (global_label "Middle" (shape input) (at 170.18 50.8 180) (fields_autoplaced)
     (effects (font (size 1.27 1.27)) (justify right))
@@
     )
   )
+  (global_label "Batt+" (shape input) (at 124.46 185.42 180) (fields_autoplaced)
+    (effects (font (size 1.27 1.27)) (justify right))
+    (property "Intersheetrefs" "${INTERSHEET_REFS}" (at 116.032 185.42 0)
+      (effects (font (size 1.27 1.27)) (justify right) hide)
+    )
+  )
+  (global_label "ADC1_BAT" (shape input) (at 190.5 66.04 0) (fields_autoplaced)
+    (effects (font (size 1.27 1.27)) (justify left))
+    (property "Intersheetrefs" "${INTERSHEET_REFS}" (at 202.6171 66.04 0)
+      (effects (font (size 1.27 1.27)) (justify left) hide)
+    )
+  )
   (global_label "Right" (shape input) (at 170.18 53.34 180) (fields_autoplaced)
     (effects (font (size 1.27 1.27)) (justify right))
@@
       (effects (font (size 1.27 1.27)) (justify left))
     )
-    (property "Footprint" "Resistor_SMD:R_0402_1005Metric" (at 175.26 120.142 90)
+    (property "Footprint" "Resistor_SMD:R_0603_1608Metric" (at 175.26 120.142 90)
       (effects (font (size 1.27 1.27)) hide)
     )
@@
       (effects (font (size 1.27 1.27)) (justify right))
     )
-    (property "Footprint" "Capacitor_SMD:C_0402_1005Metric" (at 222.5548 121.92 0)
+    (property "Footprint" "Capacitor_SMD:C_0603_1608Metric" (at 222.5548 121.92 0)
       (effects (font (size 1.27 1.27)) hide)
     )
@@
       (effects (font (size 1.27 1.27)) (justify left))
     )
-    (property "Footprint" "Resistor_SMD:R_0402_1005Metric" (at 233.172 129.54 90)
+    (property "Footprint" "Resistor_SMD:R_0603_1608Metric" (at 233.172 129.54 90)
       (effects (font (size 1.27 1.27)) hide)
     )
@@
       (effects (font (size 1.27 1.27)) (justify right))
     )
-    (property "Footprint" "LED_SMD:LED_0603_1608Metric" (at 233.68 116.84 0)
+    (property "Footprint" "LED_SMD:LED_0805_2012Metric" (at 233.68 116.84 0)
       (effects (font (size 1.27 1.27)) hide)
     )
@@
       (effects (font (size 1.27 1.27)) (justify right))
     )
-    (property "Footprint" "Capacitor_SMD:C_0402_1005Metric" (at 61.2648 49.53 0)
+    (property "Footprint" "Capacitor_SMD:C_0603_1608Metric" (at 61.2648 49.53 0)
       (effects (font (size 1.27 1.27)) hide)
     )
@@
       (effects (font (size 1.27 1.27)) (justify left))
     )
-    (property "Footprint" "Resistor_SMD:R_0402_1005Metric" (at 180.848 130.81 90)
+    (property "Footprint" "Resistor_SMD:R_0603_1608Metric" (at 180.848 130.81 90)
       (effects (font (size 1.27 1.27)) hide)
     )
@@
       (effects (font (size 1.27 1.27)) (justify right))
     )
-    (property "Footprint" "Capacitor_SMD:C_0402_1005Metric" (at 76.5048 49.53 0)
+    (property "Footprint" "Capacitor_SMD:C_0603_1608Metric" (at 76.5048 49.53 0)
       (effects (font (size 1.27 1.27)) hide)
     )
@@
       (effects (font (size 1.27 1.27)) (justify left))
     )
-    (property "Footprint" "Resistor_SMD:R_0402_1005Metric" (at 242.57 111.252 90)
+    (property "Footprint" "Resistor_SMD:R_0603_1608Metric" (at 242.57 111.252 90)
       (effects (font (size 1.27 1.27)) hide)
     )
@@
     )
   )
+  (symbol (lib_id "Device:R") (at 139.7 179.07 180) (unit 1)
+    (in_bom yes) (on_board yes) (dnp no)
+    (property "Reference" "R9" (at 137.922 180.2384 0)
+      (effects (font (size 1.27 1.27)) (justify left))
+    )
+    (property "Value" "20k" (at 137.922 177.927 0)
+      (effects (font (size 1.27 1.27)) (justify left))
+    )
+    (property "Footprint" "Resistor_SMD:R_0603_1608Metric" (at 141.478 179.07 90)
+      (effects (font (size 1.27 1.27)) hide)
+    )
+    (property "Datasheet" "~" (at 139.7 179.07 0)
+      (effects (font (size 1.27 1.27)) hide)
+    )
+    (property "JLCPN" "C4109" (at 139.7 179.07 0)
+      (effects (font (size 1.27 1.27)) hide)
+    )
+    (pin "1")
+    (pin "2")
+    (instances
+      (project "uLabel_v0"
+        (path "/531dcaa5-0d01-4877-a828-d5445ad753bd"
+          (reference "R9") (unit 1)
+        )
+      )
+      (project "ThinkTankTimerVote"
+        (path "/f5106d17-538e-4380-9554-aa558f4a587a"
+          (reference "R6") (unit 1)
+        )
+      )
+    )
+  )
+  (symbol (lib_id "Device:R") (at 124.46 179.07 0) (unit 1)
+    (in_bom yes) (on_board yes) (dnp no)
+    (property "Reference" "R9" (at 126.238 177.9016 0)
+      (effects (font (size 1.27 1.27)) (justify left))
+    )
+    (property "Value" "10k" (at 126.238 180.213 0)
+      (effects (font (size 1.27 1.27)) (justify left))
+    )
+    (property "Footprint" "Resistor_SMD:R_0603_1608Metric" (at 122.682 179.07 90)
+      (effects (font (size 1.27 1.27)) hide)
+    )
+    (property "Datasheet" "~" (at 124.46 179.07 0)
+      (effects (font (size 1.27 1.27)) hide)
+    )
+    (property "JLCPN" "C4109" (at 124.46 179.07 0)
+      (effects (font (size 1.27 1.27)) hide)
+    )
+    (pin "1")
+    (pin "2")
+    (instances
+      (project "uLabel_v0"
+        (path "/531dcaa5-0d01-4877-a828-d5445ad753bd"
+          (reference "R9") (unit 1)
+        )
+      )
+      (project "ThinkTankTimerVote"
+        (path "/f5106d17-538e-4380-9554-aa558f4a587a"
+          (reference "R5") (unit 1)
+        )
+      )
+    )
+  )
   (symbol (lib_id "Transistor_FET:IRLML2060") (at 184.15 121.92 0) (unit 1)
     (in_bom yes) (on_board yes) (dnp no) (fields_autoplaced)
@@
         )
       )
+    )
+  )
+  (symbol (lib_id "power:GND") (at 139.7 182.88 0) (unit 1)
+    (in_bom yes) (on_board yes) (dnp no) (fields_autoplaced)
+    (property "Reference" "#PWR019" (at 139.7 189.23 0)
+      (effects (font (size 1.27 1.27)) hide)
+    )
+    (property "Value" "GND" (at 139.7 187.96 0)
+      (effects (font (size 1.27 1.27)))
+    )
+    (property "Footprint" "" (at 139.7 182.88 0)
+      (effects (font (size 1.27 1.27)) hide)
+    )
+    (property "Datasheet" "" (at 139.7 182.88 0)
+      (effects (font (size 1.27 1.27)) hide)
+    )
+    (pin "1")
+    (instances
+      (project "ThinkTankTimerVote"
+        (path "/f5106d17-538e-4380-9554-aa558f4a587a"
+          (reference "#PWR019") (unit 1)
+        )
+      )
