File: TTRV PCB V5/ThinkTankTimerVote.kicad_sch (KiCad schematic)
At the start: 27 parts, among them J1 BattLeft, J2 Conn_01x02, J4 Conn_01x04, Q1 IRLML2060, SW1 SW_DPDT_x2, SW2 SW_Push, SW3 SW_Push, SW4 SW_Push, U2 HT75xx-1-SOT89, U3 LTC4054ES5-4.2

Commit message: update
Other:
- note added: "Push Buttons"
- note added: "SCREEN 128x64"
- note removed: "SSD1306 I2c"
- moved on the sheet: J4, R9

Commit message: PCB V 2.6.0
Parts:
- added J3: Conn_02x03_Odd_Even, Connector_PinHeader_2.54mm:PinHeader_2x03_P2.54mm_Vertical, symbol Connector_Generic:Conn_02x03_Odd_Even
Connections:
- net +3V3: now also J3.2 (Pin_2)
- net ADC2: now also J3.4 (Pin_4)
- net ADC3: now also J3.6 (Pin_6)
- net GND: now also J3.1 (Pin_1)
- net GPIO10: now reaches U1.10 (GPIO10)
- net GPIO10: now also J3.3 (Pin_3)
- net GPIO20: now reaches U1.20 (GPIO20)
- net GPIO20: now also J3.5 (Pin_5)
- net Motor- renamed MotorGND
Changed lines of the file:
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@@
+    (stroke (width 0) (type default))
+  )
+  (wire (pts (xy 19.05 107.95) (xy 33.02 107.95))
     (stroke (width 0) (type default))
   )
@@
   )
   (wire (pts (xy 158.75 105.41) (xy 161.29 105.41))
+    (stroke (width 0) (type default))
+  )
+  (wire (pts (xy 50.8 107.95) (xy 45.72 107.95))
     (stroke (width 0) (type default))
   )
@@
     )
   )
+  (global_label "GPIO10" (shape input) (at 33.02 110.49 180) (fields_autoplaced)
+    (effects (font (size 1.27 1.27)) (justify right))
+    (property "Intersheetrefs" "${INTERSHEET_REFS}" (at 23.1405 110.49 0)
+      (effects (font (size 1.27 1.27)) (justify right) hide)
+    )
+  )
   (global_label "ADC1_BAT" (shape input) (at 119.38 139.7 0) (fields_autoplaced)
     (effects (font (size 1.27 1.27)) (justify left))
@@
     )
   )
+  (global_label "ADC2" (shape input) (at 45.72 110.49 0) (fields_autoplaced)
+    (effects (font (size 1.27 1.27)) (justify left))
+    (property "Intersheetrefs" "${INTERSHEET_REFS}" (at 53.5433 110.49 0)
+      (effects (font (size 1.27 1.27)) (justify left) hide)
+    )
+  )
   (global_label "VILDO" (shape input) (at 95.25 49.53 180) (fields_autoplaced)
     (effects (font (size 1.27 1.27)) (justify right))
@@
     )
   )
+  (global_label "ADC3" (shape input) (at 45.72 113.03 0) (fields_autoplaced)
+    (effects (font (size 1.27 1.27)) (justify left))
+    (property "Intersheetrefs" "${INTERSHEET_REFS}" (at 53.5433 113.03 0)
+      (effects (font (size 1.27 1.27)) (justify left) hide)
+    )
+  )
   (global_label "Left" (shape input) (at 77.47 107.95 0) (fields_autoplaced)
     (effects (font (size 1.27 1.27)) (justify left))
@@
     )
   )
+  (global_label "GPIO10" (shape input) (at 170.18 63.5 180) (fields_autoplaced)
+    (effects (font (size 1.27 1.27)) (justify right))
+    (property "Intersheetrefs" "${INTERSHEET_REFS}" (at 160.3005 63.5 0)
+      (effects (font (size 1.27 1.27)) (justify right) hide)
+    )
+  )
   (global_label "Right" (shape input) (at 170.18 53.34 180) (fields_autoplaced)
     (effects (font (size 1.27 1.27)) (justify right))
@@
     )
   )
-  (global_label "Motor-" (shape input) (at 193.04 116.84 0) (fields_autoplaced)
-    (effects (font (size 1.27 1.27)) (justify left))
-    (property "Intersheetrefs" "${INTERSHEET_REFS}" (at 202.8589 116.84 0)
+  (global_label "MotorGND" (shape input) (at 193.04 116.84 0) (fields_autoplaced)
+    (effects (font (size 1.27 1.27)) (justify left))
+    (property "Intersheetrefs" "${INTERSHEET_REFS}" (at 205.157 116.84 0)
       (effects (font (size 1.27 1.27)) (justify left) hide)
     )
@@
     )
   )
+  (global_label "GPIO20" (shape input) (at 33.02 113.03 180) (fields_autoplaced)
+    (effects (font (size 1.27 1.27)) (justify right))
+    (property "Intersheetrefs" "${INTERSHEET_REFS}" (at 23.1405 113.03 0)
+      (effects (font (size 1.27 1.27)) (justify right) hide)
+    )
+  )
   (global_label "ADC2" (shape input) (at 190.5 63.5 0) (fields_autoplaced)
     (effects (font (size 1.27 1.27)) (justify left))
@@
     )
   )
-  (global_label "Motor-" (shape input) (at 160.02 113.03 180) (fields_autoplaced)
-    (effects (font (size 1.27 1.27)) (justify right))
-    (property "Intersheetrefs" "${INTERSHEET_REFS}" (at 150.2011 113.03 0)
+  (global_label "GPIO20" (shape input) (at 170.18 66.04 180) (fields_autoplaced)
+    (effects (font (size 1.27 1.27)) (justify right))
+    (property "Intersheetrefs" "${INTERSHEET_REFS}" (at 160.3005 66.04 0)
+      (effects (font (size 1.27 1.27)) (justify right) hide)
+    )
+  )
+  (global_label "MotorGND" (shape input) (at 160.02 113.03 180) (fields_autoplaced)
+    (effects (font (size 1.27 1.27)) (justify right))
+    (property "Intersheetrefs" "${INTERSHEET_REFS}" (at 147.903 113.03 0)
       (effects (font (size 1.27 1.27)) (justify right) hide)
     )
@@
     )
   )
+  (symbol (lib_id "power:+3V3") (at 50.8 107.95 0) (unit 1)
+    (in_bom yes) (on_board yes) (dnp no) (fields_autoplaced)
+    (property "Reference" "#PWR02" (at 50.8 111.76 0)
+      (effects (font (size 1.27 1.27)) hide)
+    )
+    (property "Value" "+3V3" (at 50.8 102.87 0)
+      (effects (font (size 1.27 1.27)))
+    )
+    (property "Footprint" "" (at 50.8 107.95 0)
+      (effects (font (size 1.27 1.27)) hide)
+    )
+    (property "Datasheet" "" (at 50.8 107.95 0)
+      (effects (font (size 1.27 1.27)) hide)
+    )
+    (pin "1")
+    (instances
+      (project "OM-EPSC3-Micro"
+        (path "/c7fe26ae-9505-4931-9cd8-090fc73447cd"
+          (reference "#PWR02") (unit 1)
+        )
+      )
+      (project "LASK5"
+        (path "/f2c1fb6a-8426-42c4-8a46-0c2e9dae6c65"
+          (reference "#PWR021") (unit 1)
+        )
+      )
+      (project "ThinkTankTimerVote"
+        (path "/f5106d17-538e-4380-9554-aa558f4a587a"
+          (reference "#PWR011") (unit 1)
+        )
+      )
+    )
+  )
   (symbol (lib_id "power:GND") (at 223.52 129.54 0) (unit 1)
     (in_bom yes) (on_board yes) (dnp no) (fields_autoplaced)
@@
         )
       )
+    )
+  )
+  (symbol (lib_id "power:GND") (at 19.05 107.95 0) (unit 1)
+    (in_bom yes) (on_board yes) (dnp no) (fields_autoplaced)
+    (property "Reference" "#PWR08" (at 19.05 114.3 0)
+      (effects (font (size 1.27 1.27)) hide)
+    )
+    (property "Value" "GND" (at 19.05 113.03 0)
+      (effects (font (size 1.27 1.27)))
+    )
+    (property "Footprint" "" (at 19.05 107.95 0)
+      (effects (font (size 1.27 1.27)) hide)
+    )
+    (property "Datasheet" "" (at 19.05 107.95 0)
+      (effects (font (size 1.27 1.27)) hide)
+    )
+    (pin "1")
+    (instances
+      (project "OM-EPSC3-Micro"
+        (path "/c7fe26ae-9505-4931-9cd8-090fc73447cd"
+          (reference "#PWR08") (unit 1)
+        )
+      )
+      (project "LASK5"
+        (path "/f2c1fb6a-8426-42c4-8a46-0c2e9dae6c65"
+          (reference "#PWR020") (unit 1)
+        )
+      )
+      (project "ThinkTankTimerVote"
+        (path "/f5106d17-538e-4380-9554-aa558f4a587a"
+          (reference "#PWR02") (unit 1)
+        )
+      )
+    )
+  )
+  (symbol (lib_id "Connector_Generic:Conn_02x03_Odd_Even") (at 38.1 110.49 0) (unit 1)
+    (in_bom yes) (on_board yes) (dnp no) (fields_autoplaced)
+    (property "Reference" "J3" (at 39.37 101.6 0)
+      (effects (font (size 1.27 1.27)))
+    )
+    (property "Value" "Conn_02x03_Odd_Even" (at 39.37 104.14 0)
+      (effects (font (size 1.27 1.27)))
+    )
+    (property "Footprint" "Connector_PinHeader_2.54mm:PinHeader_2x03_P2.54mm_Vertical" (at 38.1 110.49 0)
+      (effects (font (size 1.27 1.27)) hide)
+    )
+    (property "Datasheet" "~" (at 38.1 110.49 0)
+      (effects (font (size 1.27 1.27)) hide)
+    )
+    (pin "1")
+    (pin "2")
+    (pin "3")
+    (pin "4")
+    (pin "5")
+    (pin "6")
+    (instances
+      (project "ThinkTankTimerVote"
+        (path "/f5106d17-538e-4380-9554-aa558f4a587a"
+          (reference "J3") (unit 1)
+        )
+      )

Commit message: v2.1 updates
Parts:
- R9: value 2k -> 150
Connections:
- net +5V: now also R9.1, U3.4 (V_{CC}); no longer D2.2 (A), R9.2
- new net: D2.2 (A), R9.2
Other:
- moved on the sheet: D2
Changed lines of the file:
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@@
 (kicad_sch (version 20230121) (generator eeschema)
   (paper "A4")
+  (junction (at 243.84 113.03) (diameter 0) (color 0 0 0 0)
+  )
   (junction (at 186.69 134.62) (diameter 0) (color 0 0 0 0)
   )
@@
   (junction (at 161.29 113.03) (diameter 0) (color 0 0 0 0)
   )
-  (junction (at 233.68 113.03) (diameter 0) (color 0 0 0 0)
-  )
   (junction (at 173.99 113.03) (diameter 0) (color 0 0 0 0)
   )
@@
     (stroke (width 0) (type default))
   )
+  (wire (pts (xy 241.3 115.57) (xy 243.84 115.57))
+    (stroke (width 0) (type default))
+  )
   (wire (pts (xy 251.46 46.99) (xy 246.38 46.99))
     (stroke (width 0) (type default))
@@
     (stroke (width 0) (type default))
   )
-  (wire (pts (xy 223.52 113.03) (xy 233.68 113.03))
-    (stroke (width 0) (type default))
-  )
   (wire (pts (xy 186.69 135.89) (xy 186.69 134.62))
     (stroke (width 0) (type default))
@@
     (stroke (width 0) (type default))
   )
+  (wire (pts (xy 243.84 115.57) (xy 243.84 113.03))
+    (stroke (width 0) (type default))
+  )
   (wire (pts (xy 125.73 113.03) (xy 121.92 113.03))
     (stroke (width 0) (type default))
@@
     (stroke (width 0) (type default))
   )
+  (wire (pts (xy 243.84 113.03) (xy 250.19 113.03))
+    (stroke (width 0) (type default))
+  )
   (wire (pts (xy 227.33 54.61) (xy 236.22 54.61))
     (stroke (width 0) (type default))
@@
     (stroke (width 0) (type default))
   )
-  (wire (pts (xy 233.68 113.03) (xy 238.76 113.03))
-    (stroke (width 0) (type default))
-  )
-  (wire (pts (xy 233.68 120.65) (xy 233.68 123.19))
-    (stroke (width 0) (type default))
-  )
   (wire (pts (xy 234.95 125.73) (xy 240.03 125.73))
     (stroke (width 0) (type default))
   )
-  (wire (pts (xy 246.38 113.03) (xy 250.19 113.03))
+  (wire (pts (xy 223.52 113.03) (xy 243.84 113.03))
     (stroke (width 0) (type default))
   )
@@
     )
   )
-  (symbol (lib_id "Device:LED") (at 233.68 116.84 90) (unit 1)
+  (symbol (lib_id "Device:LED") (at 233.68 119.38 90) (unit 1)
     (in_bom yes) (on_board yes) (dnp no)
-    (property "Reference" "D2" (at 236.6518 115.8748 90)
+    (property "Reference" "D2" (at 226.06 116.84 90)
       (effects (font (size 1.27 1.27)) (justify right))
     )
-    (property "Value" "LED GREEN" (at 231.14 113.03 0)
+    (property "Value" "LED GREEN" (at 231.14 115.57 0)
       (effects (font (size 1.27 1.27)) (justify right))
     )
-    (property "Footprint" "LED_SMD:LED_0805_2012Metric" (at 233.68 116.84 0)
-      (effects (font (size 1.27 1.27)) hide)
-    )
-    (property "Datasheet" "~" (at 233.68 116.84 0)
-      (effects (font (size 1.27 1.27)) hide)
-    )
-    (property "JLCPN" "C72043" (at 233.68 116.84 90)
+    (property "Footprint" "LED_SMD:LED_0805_2012Metric" (at 233.68 119.38 0)
+      (effects (font (size 1.27 1.27)) hide)
+    )
+    (property "Datasheet" "~" (at 233.68 119.38 0)
+      (effects (font (size 1.27 1.27)) hide)
+    )
+    (property "JLCPN" "C72043" (at 233.68 119.38 90)
       (effects (font (size 1.27 1.27)) hide)
     )
@@
     )
   )
+  (symbol (lib_id "Device:R") (at 237.49 115.57 270) (unit 1)
+    (in_bom yes) (on_board yes) (dnp no)
+    (property "Reference" "R9" (at 238.6584 117.348 0)
+      (effects (font (size 1.27 1.27)) (justify left))
+    )
+    (property "Value" "150" (at 236.22 116.84 0)
+      (effects (font (size 1.27 1.27)) (justify left))
+    )
+    (property "Footprint" "Resistor_SMD:R_0603_1608Metric" (at 237.49 113.792 90)
+      (effects (font (size 1.27 1.27)) hide)
+    )
+    (property "Datasheet" "~" (at 237.49 115.57 0)
+      (effects (font (size 1.27 1.27)) hide)
+    )
+    (property "JLCPN" "C4109" (at 237.49 115.57 0)
+      (effects (font (size 1.27 1.27)) hide)
+    )
+    (pin "1")
+    (pin "2")
+    (instances
+      (project "uLabel_v0"
+        (path "/531dcaa5-0d01-4877-a828-d5445ad753bd"
+          (reference "R9") (unit 1)
+        )
+      )
+      (project "ThinkTankTimerVote"
+        (path "/f5106d17-538e-4380-9554-aa558f4a587a"
+          (reference "R3") (unit 1)
+        )
+      )
+    )
+  )
   (symbol (lib_id "power:GND") (at 19.05 107.95 0) (unit 1)
     (in_bom yes) (on_board yes) (dnp no) (fields_autoplaced)
@@
         )
       )
-    )
-  )
-  (symbol (lib_id "Device:R") (at 242.57 113.03 270) (unit 1)
-    (in_bom yes) (on_board yes) (dnp no)
-    (property "Reference" "R9" (at 243.7384 114.808 0)
-      (effects (font (size 1.27 1.27)) (justify left))
-    )
-    (property "Value" "2k" (at 241.427 114.808 0)
-      (effects (font (size 1.27 1.27)) (justify left))
-    )
-    (property "Footprint" "Resistor_SMD:R_0603_1608Metric" (at 242.57 111.252 90)
-      (effects (font (size 1.27 1.27)) hide)
-    )
-    (property "Datasheet" "~" (at 242.57 113.03 0)
-      (effects (font (size 1.27 1.27)) hide)
-    )
-    (property "JLCPN" "C4109" (at 242.57 113.03 0)
-      (effects (font (size 1.27 1.27)) hide)
-    )
-    (pin "1")
-    (pin "2")
-    (instances
-      (project "uLabel_v0"
-        (path "/531dcaa5-0d01-4877-a828-d5445ad753bd"
-          (reference "R9") (unit 1)
-        )
-      )
-      (project "ThinkTankTimerVote"
-        (path "/f5106d17-538e-4380-9554-aa558f4a587a"
-          (reference "R3") (unit 1)
-        )
-      )
